File: sch/rusty-hangulclock/rusty-hangulclock.kicad_pcb (KiCad board)
At the start: 2 copper layers, 45 x 54 mm, 15 parts, among them J1 Conn_OLED, J2 Conn_SLEDS, J3 PWR, SW1 RotaryEncoder_Switch_MP, U1 74AHCT125

Commit message: update sch
Parts:
- added C5: 100n, Capacitor_THT:C_Disc_D5.0mm_W2.5mm_P5.00mm, F.Cu at (135.2, 95.0)
- moved C2 2.00 mm to (135.2, 92.0)
Routing:
- net +5V: track 58.4 -> 62.4 mm
- net Net-(ESP32-C3_SuperMini1-P1): track 36.5 -> 38.6 mm
Changed lines of the file:
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@@
 	(footprint "Capacitor_THT:C_Disc_D5.0mm_W2.5mm_P5.00mm"
 		(layer "F.Cu")
+		(at 135.25 95 180)
+		(descr "C, Disc series, Radial, pin pitch=5.00mm, diameter*width=5*2.5mm^2, Capacitor, http://cdn-reichelt.de/documents/datenblatt/B300/DS_KERKO_TC.pdf")
+		(tags "C Disc series Radial pin pitch 5.00mm diameter 5mm width 2.5mm Capacitor")
+		(property "Reference" "C5"
+			(at 2.5 -2.5 0)
+			(layer "F.SilkS")
+			(effects
+				(font
+					(size 1 1)
+					(thickness 0.15)
+				)
+			)
+		)
+		(property "Value" "100n"
+			(at 2.5 2.5 0)
+			(layer "F.Fab")
+			(effects
+				(font
+					(size 1 1)
+					(thickness 0.15)
+				)
+			)
+		)
+		(property "Datasheet" ""
+			(at 0 0 0)
+			(layer "F.Fab")
+			(hide yes)
+			(effects
+				(font
+					(size 1.27 1.27)
+					(thickness 0.15)
+				)
+			)
+		)
+		(property "Description" "Unpolarized capacitor"
+			(at 0 0 0)
+			(layer "F.Fab")
+			(hide yes)
+			(effects
+				(font
+					(size 1.27 1.27)
+					(thickness 0.15)
+				)
+			)
+		)
+		(property ki_fp_filters "C_*")
+		(sheetname "/")
+		(sheetfile "rusty-hangulclock.kicad_sch")
+		(attr through_hole)
+		(fp_line
+			(start 5.12 1.033)
+			(end 5.12 1.37)
+			(stroke
+				(width 0.12)
+				(type solid)
+			)
+			(layer "F.SilkS")
+		)
+		(fp_line
+			(start 5.12 -1.37)
+			(end 5.12 -1.033)
+			(stroke
+				(width 0.12)
+				(type solid)
+			)
+			(layer "F.SilkS")
+		)
+		(fp_line
+			(start -0.12 1.37)
+			(end 5.12 1.37)
+			(stroke
+				(width 0.12)
+				(type solid)
+			)
+			(layer "F.SilkS")
+		)
+		(fp_line
+			(start -0.12 1.033)
+			(end -0.12 1.37)
+			(stroke
+				(width 0.12)
+				(type solid)
+			)
+			(layer "F.SilkS")
+		)
+		(fp_line
+			(start -0.12 -1.37)
+			(end 5.12 -1.37)
+			(stroke
+				(width 0.12)
+				(type solid)
+			)
+			(layer "F.SilkS")
+		)
+		(fp_line
+			(start -0.12 -1.37)
+			(end -0.12 -1.033)
+			(stroke
+				(width 0.12)
+				(type solid)
+			)
+			(layer "F.SilkS")
+		)
+		(fp_rect
+			(start -1.05 -1.5)
+			(end 6.05 1.5)
+			(stroke
+				(width 0.05)
+				(type solid)
+			)
+			(fill no)
+			(layer "F.CrtYd")
+		)
+		(fp_rect
+			(start 0 -1.25)
+			(end 5 1.25)
+			(stroke
+				(width 0.1)
+				(type solid)
+			)
+			(fill no)
+			(layer "F.Fab")
+		)
+		(fp_text user "${REFERENCE}"
+			(at 2.5 0 0)
+			(layer "F.Fab")
+			(effects
+				(font
+					(size 1 1)
+					(thickness 0.15)
+				)
+			)
+		)
+		(pad "1" thru_hole circle
+			(at 0 0 180)
+			(size 1.6 1.6)
+			(drill 0.8)
+			(layers "*.Cu" "*.Mask")
+			(remove_unused_layers no)
+			(net 5 "+5V")
+			(pintype "passive")
+		)
+		(pad "2" thru_hole circle
+			(at 5 0 180)
+			(size 1.6 1.6)
+			(drill 0.8)
+			(layers "*.Cu" "*.Mask")
+			(remove_unused_layers no)
+			(net 1 "GND")
+			(pintype "passive")
+		)
+		(embedded_fonts no)
+		(model "${KICAD9_3DMODEL_DIR}/Capacitor_THT.3dshapes/C_Disc_D5.0mm_W2.5mm_P5.00mm.step"
+			(offset
+				(xyz 0 0 0)
+			)
+			(scale
+				(xyz 1 1 1)
+			)
+			(rotate
+				(xyz 0 0 0)
+			)
+		)
+	)
+	(footprint "Capacitor_THT:C_Disc_D5.0mm_W2.5mm_P5.00mm"
+		(layer "F.Cu")
 		(at 159 98.5 90)
 		(descr "C, Disc series, Radial, pin pitch=5.00mm, , diameter*width=5*2.5mm^2, Capacitor, http://cdn-reichelt.de/documents/datenblatt/B300/DS_KERKO_TC.pdf")
@@
 	(footprint "Capacitor_THT:C_Disc_D5.0mm_W2.5mm_P5.00mm"
 		(layer "F.Cu")
-		(at 135.25 94 180)
+		(at 135.25 92 180)
 		(descr "C, Disc series, Radial, pin pitch=5.00mm, , diameter*width=5*2.5mm^2, Capacitor, http://cdn-reichelt.de/documents/datenblatt/B300/DS_KERKO_TC.pdf")
 		(tags "C Disc series Radial pin pitch 5.00mm  diameter 5mm width 2.5mm Capacitor")
@@
 	)
 	(segment
+		(start 134.31 95.94)
+		(end 135.25 95)
+		(width 0.5)
+		(layer "B.Cu")
+		(net 5)
+	)
+	(segment
 		(start 124 112)
 		(end 124 102.5)
@@
 	)
 	(segment
+		(start 134.31 98.525)
+		(end 134.31 95.94)
+		(width 0.5)
+		(layer "B.Cu")
+		(net 5)
+	)
+	(segment
 		(start 133 101)
 		(end 134.31 99.69)
@@
 	(segment
 		(start 135.25 121.17)
-		(end 135.25 94)
+		(end 135.25 103.25)
 		(width 0.2)
 		(layer "F.Cu")
@@
 	)
 	(segment
-		(start 139.75 96.25)
-		(end 137.25 96.25)
+		(start 139.75 98.75)
+		(end 139.75 96.25)
 		(width 0.2)
 		(layer "F.Cu")
@@
 	)
 	(segment
-		(start 136.5 95.25)
-		(end 135.25 94)
+		(start 137 95.5)
+		(end 137 92.5)
 		(width 0.2)
 		(layer "F.Cu")
@@
 	)
 	(segment
-		(start 138.5 122.42)
-		(end 136.5 122.42)
+		(start 137.75 96.25)
+		(end 137 95.5)
 		(width 0.2)
 		(layer "F.Cu")
@@
 	)
 	(segment
-		(start 136.5 95.5)
-		(end 136.5 95.25)
+		(start 136.5 122.42)
+		(end 135.25 121.17)
 		(width 0.2)
 		(layer "F.Cu")
@@
 	)
 	(segment
-		(start 137.25 96.25)
-		(end 136.5 95.5)
+		(start 139.75 96.25)
+		(end 137.75 96.25)
 		(width 0.2)
 		(layer "F.Cu")
@@
 	)
 	(segment
-		(start 136.5 122.42)
-		(end 135.25 121.17)
+		(start 137 92.5)
+		(end 136.5 92)
+		(width 0.2)
+		(layer "F.Cu")
+		(net 6)
+	)
+	(segment
+		(start 135.25 103.25)
+		(end 139.75 98.75)
+		(width 0.2)
+		(layer "F.Cu")
+		(net 6)
+	)
+	(segment
+		(start 138.5 122.42)
+		(end 136.5 122.42)
+		(width 0.2)
+		(layer "F.Cu")
+		(net 6)
+	)
+	(segment
+		(start 136.5 92)
+		(end 135.25 92)
 		(width 0.2)
 		(layer "F.Cu")

Commit message: fixing
Parts:
- removed ESP32-C3_SuperMini1: ~, Homin_Library:ESP32-C3_SuperMini_SMD
- removed G***: LOGO, LOGO
- removed U1: 74AHCT125, Package_SO:SOIC-14_3.9x8.7mm_P1.27mm
- added C10: 100n, Capacitor_SMD:C_0805_2012Metric_Pad1.18x1.45mm_HandSolder, F.Cu at (341.6, 55.1)
- added C11: 100n, Capacitor_SMD:C_0805_2012Metric_Pad1.18x1.45mm_HandSolder, F.Cu at (341.6, 59.2)
- added C12: 100n, Capacitor_SMD:C_0805_2012Metric_Pad1.18x1.45mm_HandSolder, F.Cu at (341.6, 63.2)
- added C13: 100n, Capacitor_SMD:C_0805_2012Metric_Pad1.18x1.45mm_HandSolder, F.Cu at (341.6, 67.3)
- added C14: 100n, Capacitor_SMD:C_0805_2012Metric_Pad1.18x1.45mm_HandSolder, F.Cu at (341.6, 71.3)
- added C15: 100n, Capacitor_SMD:C_0805_2012Metric_Pad1.18x1.45mm_HandSolder, F.Cu at (341.6, 75.4)
- added C16: 100n, Capacitor_SMD:C_0805_2012Metric_Pad1.18x1.45mm_HandSolder, F.Cu at (341.6, 79.5)
- added C17: 100n, Capacitor_SMD:C_0805_2012Metric_Pad1.18x1.45mm_HandSolder, F.Cu at (341.6, 83.5)
- added C18: 100n, Capacitor_SMD:C_0805_2012Metric_Pad1.18x1.45mm_HandSolder, F.Cu at (349.8, 55.1)
- added C19: 100n, Capacitor_SMD:C_0805_2012Metric_Pad1.18x1.45mm_HandSolder, F.Cu at (349.8, 59.2)
- added C20: 100n, Capacitor_SMD:C_0805_2012Metric_Pad1.18x1.45mm_HandSolder, F.Cu at (349.8, 63.2)
- added C21: 100n, Capacitor_SMD:C_0805_2012Metric_Pad1.18x1.45mm_HandSolder, F.Cu at (349.8, 67.3)
- added C22: 100n, Capacitor_SMD:C_0805_2012Metric_Pad1.18x1.45mm_HandSolder, F.Cu at (349.8, 71.3)
- added C23: 100n, Capacitor_SMD:C_0805_2012Metric_Pad1.18x1.45mm_HandSolder, F.Cu at (349.8, 75.4)
- added C24: 100n, Capacitor_SMD:C_0805_2012Metric_Pad1.18x1.45mm_HandSolder, F.Cu at (349.8, 79.5)
- added C25: 100n, Capacitor_SMD:C_0805_2012Metric_Pad1.18x1.45mm_HandSolder, F.Cu at (349.8, 83.5)
- added C26: 100n, Capacitor_SMD:C_0805_2012Metric_Pad1.18x1.45mm_HandSolder, F.Cu at (357.9, 55.1)
- added C27: 100n, Capacitor_SMD:C_0805_2012Metric_Pad1.18x1.45mm_HandSolder, F.Cu at (357.9, 59.2)
- added C28: 100n, Capacitor_SMD:C_0805_2012Metric_Pad1.18x1.45mm_HandSolder, F.Cu at (357.9, 63.2)
- added C29: 100n, Capacitor_SMD:C_0805_2012Metric_Pad1.18x1.45mm_HandSolder, F.Cu at (357.9, 67.3)
- added C30: 100n, Capacitor_SMD:C_0805_2012Metric_Pad1.18x1.45mm_HandSolder, F.Cu at (357.9, 71.3)
- added C31: 100n, Capacitor_SMD:C_0805_2012Metric_Pad1.18x1.45mm_HandSolder, F.Cu at (357.9, 75.4)
- added C6: 100n, Capacitor_SMD:C_0805_2012Metric_Pad1.18x1.45mm_HandSolder, F.Cu at (333.4, 71.3)
- added C7: 100n, Capacitor_SMD:C_0805_2012Metric_Pad1.18x1.45mm_HandSolder, F.Cu at (333.4, 75.4)
- added C8: 100n, Capacitor_SMD:C_0805_2012Metric_Pad1.18x1.45mm_HandSolder, F.Cu at (333.4, 79.5)
- added C9: 100n, Capacitor_SMD:C_0805_2012Metric_Pad1.18x1.45mm_HandSolder, F.Cu at (333.4, 83.5)
- added D1: WS2812B, LED_SMD:LED_WS2812B_PLCC4_5.0x5.0mm_P3.2mm, F.Cu at (335.9, 23.3)
- added D10: WS2812B, LED_SMD:LED_WS2812B_PLCC4_5.0x5.0mm_P3.2mm, F.Cu at (344.1, 49.8)
- added D11: WS2812B, LED_SMD:LED_WS2812B_PLCC4_5.0x5.0mm_P3.2mm, F.Cu at (352.2, 23.3)
- added D12: WS2812B, LED_SMD:LED_WS2812B_PLCC4_5.0x5.0mm_P3.2mm, F.Cu at (352.2, 30.0)
- added D13: WS2812B, LED_SMD:LED_WS2812B_PLCC4_5.0x5.0mm_P3.2mm, F.Cu at (352.2, 36.6)
- added D14: WS2812B, LED_SMD:LED_WS2812B_PLCC4_5.0x5.0mm_P3.2mm, F.Cu at (352.2, 43.2)
- added D15: WS2812B, LED_SMD:LED_WS2812B_PLCC4_5.0x5.0mm_P3.2mm, F.Cu at (352.2, 49.8)
- added D16: WS2812B, LED_SMD:LED_WS2812B_PLCC4_5.0x5.0mm_P3.2mm, F.Cu at (360.3, 23.3)
- added D17: WS2812B, LED_SMD:LED_WS2812B_PLCC4_5.0x5.0mm_P3.2mm, F.Cu at (360.3, 30.0)
- added D18: WS2812B, LED_SMD:LED_WS2812B_PLCC4_5.0x5.0mm_P3.2mm, F.Cu at (360.3, 36.6)
- added D19: WS2812B, LED_SMD:LED_WS2812B_PLCC4_5.0x5.0mm_P3.2mm, F.Cu at (360.3, 43.2)
- added D2: WS2812B, LED_SMD:LED_WS2812B_PLCC4_5.0x5.0mm_P3.2mm, F.Cu at (335.9, 30.0)
- added D20: WS2812B, LED_SMD:LED_WS2812B_PLCC4_5.0x5.0mm_P3.2mm, F.Cu at (360.3, 49.8)
- added D21: WS2812B, LED_SMD:LED_WS2812B_PLCC4_5.0x5.0mm_P3.2mm, F.Cu at (368.4, 23.3)
- added D22: WS2812B, LED_SMD:LED_WS2812B_PLCC4_5.0x5.0mm_P3.2mm, F.Cu at (368.4, 30.0)
- added D23: WS2812B, LED_SMD:LED_WS2812B_PLCC4_5.0x5.0mm_P3.2mm, F.Cu at (368.4, 36.6)
- added D24: WS2812B, LED_SMD:LED_WS2812B_PLCC4_5.0x5.0mm_P3.2mm, F.Cu at (368.4, 43.2)
- added D25: WS2812B, LED_SMD:LED_WS2812B_PLCC4_5.0x5.0mm_P3.2mm, F.Cu at (368.4, 49.8)
- added D26: D, Diode_SMD:D_0805_2012Metric, F.Cu at (391.9, 49.5)
- added D3: WS2812B, LED_SMD:LED_WS2812B_PLCC4_5.0x5.0mm_P3.2mm, F.Cu at (335.9, 36.6)
- added D4: WS2812B, LED_SMD:LED_WS2812B_PLCC4_5.0x5.0mm_P3.2mm, F.Cu at (335.9, 43.2)
- added D5: WS2812B, LED_SMD:LED_WS2812B_PLCC4_5.0x5.0mm_P3.2mm, F.Cu at (335.9, 49.8)
- added D6: WS2812B, LED_SMD:LED_WS2812B_PLCC4_5.0x5.0mm_P3.2mm, F.Cu at (344.1, 23.3)
- added D7: WS2812B, LED_SMD:LED_WS2812B_PLCC4_5.0x5.0mm_P3.2mm, F.Cu at (344.1, 30.0)
- added D8: WS2812B, LED_SMD:LED_WS2812B_PLCC4_5.0x5.0mm_P3.2mm, F.Cu at (344.1, 36.6)
- added D9: WS2812B, LED_SMD:LED_WS2812B_PLCC4_5.0x5.0mm_P3.2mm, F.Cu at (344.1, 43.2)
- added R1: 10k, Resistor_SMD:R_0805_2012Metric, F.Cu at (396.3, 49.4)
- added U2: ESP32-C3-WROOM-02, RF_Module:ESP32-C3-WROOM-02, F.Cu at (379.2, 72.0)
- C2, C3, C4, C5: footprint Capacitor_THT:C_Disc_D5.0mm_W2.5mm_P5.00mm -> Capacitor_SMD:C_0805_2012Metric_Pad1.18x1.45mm_HandSolder
- J2: value Conn_SLEDS -> Conn_OLED; footprint Connector_PinHeader_2.54mm:PinHeader_1x04_P2.54mm_Horizontal -> Connector_PinHeader_2.54mm:PinHeader_1x04_P2.54mm_Vertical
- moved J3 276.9 mm to (391.9, 37.6), turned to 0 degrees
- moved C1 272.3 mm to (391.4, 45.2), turned to 0 degrees
- moved H3 269.5 mm to (376.4, 39.9), turned to 0 degrees
- moved J2 267.6 mm to (387.3, 37.6), turned to 0 degrees
- moved H4 255.2 mm to (376.4, 47.9), turned to 0 degrees
- moved SW1 251.5 mm to (382.4, 25.1)
- moved H2 237.7 mm to (376.4, 31.9), turned to 0 degrees
- moved J1 233.1 mm to (382.7, 37.6), turned to 0 degrees
- moved H1 223.5 mm to (376.4, 24.0), turned to 0 degrees
- moved C2 201.6 mm to (333.4, 55.1), turned to 0 degrees
- moved C3 200.4 mm to (333.4, 59.2), turned to 0 degrees
- moved C5 200.1 mm to (333.4, 67.3), turned to 0 degrees
- moved C4 178.0 mm to (333.4, 63.2), turned to 0 degrees
Connections:
- J1 pad 3: Net-(ESP32-C3_SuperMini1-P9) -> Net-(J1-Pin_3)
- J1 pad 4: Net-(ESP32-C3_SuperMini1-P8) -> Net-(J1-Pin_4)
- J2 pad 1: +5V -> GND
- J2 pad 2: Net-(J2-Pin_2) -> +3V3
- J2 pad 3: Net-(J2-Pin_3) -> Net-(J1-Pin_3)
- J2 pad 4: GND -> Net-(J1-Pin_4)
Routing:
- net +5V: track 62.4 -> 0.00 mm
- net Net-(U2-IO3): track 49.9 -> 0.00 mm
- net Net-(U2-IO2): track 45.8 -> 0.00 mm
- net Net-(ESP32-C3_SuperMini1-P6): track 45.0 -> 0.00 mm, vias 1 -> 0
- net Net-(U2-IO1): track 38.6 -> 0.00 mm
- net Net-(ESP32-C3_SuperMini1-P4): track 32.2 -> 0.00 mm, vias 1 -> 0
- net +3V3: track 31.6 -> 0.00 mm, vias 1 -> 0
- net Net-(ESP32-C3_SuperMini1-P8): track 29.4 -> 0.00 mm
- net Net-(ESP32-C3_SuperMini1-P9): track 20.9 -> 0.00 mm
- net Net-(J2-Pin_3): track 11.8 -> 0.00 mm
- net Net-(J2-Pin_2): track 11.6 -> 0.00 mm
- net GND: vias 4 -> 0
- removed copper zone on B.Cu, net GND
- removed copper zone on F.Cu, net GND
Other:
- board outline removed
- board text removed: "3V3"
- board text removed: "5V"
- board text removed: "GND"
- board text removed: "P4SCK"
- board text removed: "P6MOSI"
- board text removed: "Rusty HangulClock By Homin Lee May 2025 https://github.com/suapapa /rusty-hangulclock"
- board text removed: "SCL"
- board text removed: "SDA"
