File: sch/rusty-hangulclock_rev4/rusty-hangulclock.kicad_pcb (KiCad board)
At the start: 2 copper layers, 170 x 170 mm, 91 parts, among them J1 Conn_OLED, J2 Conn_OLED, J3 Conn_USB2, J4 USB_C_Receptacle_PowerOnly_6P, Q1 S8050, SW1 RotaryEncoder_Switch_MP, U1 ESP32-C3-WROOM-02, U2 SY8088, U3 DS3231MZ

Commit message: fix: update sch
Parts:
- removed M1: ~, Library:ESP32-C3_SuperMini_THT
- R2, R6: value 56kΩ -> 5.1kΩ
- moved J1 33.0 mm to (95.5, 61.0)
- moved J2 33.0 mm to (86.5, 61.0)
- moved C35 0.25 mm to (144.0, 152.0)
- moved R7 0.25 mm to (144.0, 155.5)
Routing:
- net +5V: track 1064.1 -> 968.2 mm, vias 12 -> 11
- net +3V3: track 202.4 -> 249.4 mm
- net IO9: track 227.8 -> 190.0 mm, vias 1 -> 0
- net IO8: track 218.7 -> 185.1 mm, vias 1 -> 0
- net IO6: track 197.6 -> 164.1 mm, vias 2 -> 1
- net IO3: track 131.2 -> 102.0 mm
- net IO2: track 108.5 -> 83.5 mm
- net IO1: track 118.5 -> 93.6 mm
- net D-: track 47.7 -> 29.4 mm
- net GND: track 0.00 -> 8.71 mm, vias 28 -> 32
- net Net-(J4-SHIELD): track 12.6 -> 17.3 mm
- net EN: track 82.0 -> 85.6 mm
- net Net-(U2-FB): track 9.95 -> 12.0 mm
- net D+: track 28.8 -> 29.4 mm
Other:
- board text added: "한글시계 - RustyHangulClock Rev-4.3 (Oct. 2025) https://hangulclock.homin.dev - 설명서를 보려면 QR 코드를 스캔하세요. - 다이얼(노브)을 돌려 메뉴를 탐색하세요. - 다이얼(노브)을 눌러 메뉴 항목을 선택하거나 선택을 결정하세요. - Scan the QR code for instructions. - Turn the knob to navigate the menu. - Press the knob to select a menu item or confirm a selection."
- board text removed: "Rusty HangulClock rev.5 (June 2025) https://hangulclock.homin.dev - Scan the QR code for instructions. - Turn the knob to navigate the menu. - Press the knob to select a menu item or confirm a selection."

Commit message: fix: sch
Parts:
- removed R9: 10kΩ, PCM_JLCPCB:R_0402
- added Q2: S8050, PCM_JLCPCB:Q_SOT-23, B.Cu at (30.2, 41.8)
- added R10: 10kΩ, PCM_JLCPCB:R_0402, B.Cu at (35.8, 45.2)
- added R11: 10kΩ, PCM_JLCPCB:R_0402, B.Cu at (35.8, 48.8)
- added R5: 1kΩ, PCM_JLCPCB:R_0402, B.Cu at (35.8, 47.0)
- moved Q1 4.75 mm to (30.2, 47.0)
- moved R8 2.30 mm to (35.8, 50.5)
Connections:
- Q1 pad 2: LED_IN -> GND
- Q1 pad 3: +5V -> Net-(Q1-C)
Routing:
- net +3V3: track 249.4 -> 305.7 mm, vias 2 -> 3
- net Net-(Q2-B): track 0.00 -> 7.72 mm
- net Net-(Q1-C): track 0.00 -> 7.04 mm
- net LED_IN: track 17.1 -> 14.1 mm
- net Net-(Q1-B): track 4.06 -> 7.04 mm
- net +5V: track 968.2 -> 966.2 mm
- net IO6: track 164.1 -> 164.9 mm
